File: BMI270.kicad_pcb (KiCad board)
At the start: 2 copper layers, 18 x 13 mm, 10 parts, among them J1 Conn_01x07_Socket, J2 Conn_01x05_Socket, U1 BMI270

Commit message: Fix labels
Other:
- board text added: "J1"
Changed lines of the file:
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@@
 		(tags "resistor")
 		(property "Reference" "R3"
-			(at 3.085 0.544441 0)
+			(at 2.349 -0.15 0)
 			(layer "F.SilkS")
 			(effects
@@
 		)
 	)
+	(gr_text "J1\n"
+		(at 139.954 108.862 90)
+		(layer "F.SilkS")
+		(effects
+			(font
+				(size 1 1)
+				(thickness 0.15)
+			)
+		)
+	)
 	(gr_text "X"
 		(at 140.25 103.92 180)
@@
 	)
 	(via
-		(at 138.43 108.1)
+		(at 139.192 108.1)
 		(size 0.6)
 		(drill 0.3)
@@
 	)
 	(segment
+		(start 139.192 106.738)
+		(end 139.7 106.23)
+		(width 0.2)
+		(layer "B.Cu")
+		(net 11)
+	)
+	(segment
 		(start 139.7 107.743654)
 		(end 142.596346 110.64)
@@
 	)
 	(segment
-		(start 139.7 106.23)
-		(end 138.43 107.5)
-		(width 0.2)
-		(layer "B.Cu")
-		(net 11)
-	)
-	(segment
 		(start 145.693654 101.75)
 		(end 145.376497 101.432843)
@@
 	)
 	(segment
-		(start 138.43 107.5)
-		(end 138.43 108.1)
-		(width 0.2)
-		(layer "B.Cu")
-		(net 11)
-	)
-	(segment
 		(start 143.51 103.02)
 		(end 140.3 106.23)
 		(width 0.2)
 		(layer "B.Cu")
+		(net 11)
+	)
+	(segment
+		(start 139.192 108.1)
+		(end 139.192 106.738)
+		(width 0.2)
+		(layer "B.Cu")
